File: PCB/HighPrecPosSens.kicad_sch (KiCad schematic)
At the start: 92 parts, among them J1 Conn_01x02_Male, J2 Conn_01x02_Male, J3 Conn_01x02_Male, J4 Conn_01x02_Male, J5 Conn_01x06_Male, J6 Conn_01x02_Male, J7 Conn_01x02_Male, J8 Conn_01x02_Male, U1 ST1S14PHR, U2 S12443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

Commit message: Added logo
Parts:
- added G1: LOGO, Logos:enGyneer-Logo, symbol enGyneer-Logo:LOGO
Changed lines of the file:
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@@
     (pin "2")
+  )
+  (symbol (lib_id "enGyneer-Logo:LOGO") (at 343.535 260.35 0) (unit 1)
+    (in_bom yes) (on_board yes) (fields_autoplaced)
+    (property "Reference" "G1" (id 0) (at 346.075 256.54 0)
+      (effects (font (size 1.27 1.27)) hide)
+    )
+    (property "Value" "LOGO" (id 1) (at 343.535 265.43 0)
+      (effects (font (size 1.27 1.27)) hide)
+    )
+    (property "Footprint" "Logos:enGyneer-Logo" (id 2) (at 343.535 260.35 0)
+      (effects (font (size 1.27 1.27)) hide)
+    )
+    (property "Datasheet" "" (id 3) (at 343.535 260.35 0)
+      (effects (font (size 1.27 1.27)) hide)
+    )
+    (property "Mounting" "DNP" (id 4) (at 343.535 260.35 0)
+      (effects (font (size 1.27 1.27)) hide)
+    )
   )
   (symbol (lib_id "Device:C") (at 21.59 251.46 0) (unit 1)
@@
       (reference "FID4") (unit 1) (value "Fiducial") (footprint "Fiducial:Fiducial_1mm_Mask2mm")
     )
+    (path "/6d3764de-e6f2-4455-9559-cbfdc0358963"
+      (reference "G1") (unit 1) (value "LOGO") (footprint "Logos:enGyneer-Logo")
+    )
     (path "/cffb5fac-e82d-404f-bf3f-17054244c031"

Commit message: changed vias
Parts:
- J5: Manufacturer (none) -> JST; ManufacturerPartNum (none) -> B6B-XH-A(LF)(SN); Sourcing (none) -> JLCPCB; SourcingPartNum (none) -> C144397
Changed lines of the file:
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@@
       (effects (font (size 1.27 1.27)) hide)
     )
-    (property "Datasheet" "~" (id 3) (at 116.84 193.04 0)
+    (property "Datasheet" "https://datasheet.lcsc.com/lcsc/1810291333_JST-Sales-America-B6B-XH-A-LF-SN_C144397.pdf" (id 3) (at 116.84 193.04 0)
       (effects (font (size 1.27 1.27)) hide)
     )
@@
       (effects (font (size 1.27 1.27)) hide)
     )
+    (property "Manufacturer" "JST" (id 5) (at 116.84 193.04 0)
+      (effects (font (size 1.27 1.27)) hide)
+    )
+    (property "ManufacturerPartNum" "B6B-XH-A(LF)(SN)" (id 6) (at 116.84 193.04 0)
+      (effects (font (size 1.27 1.27)) hide)
+    )
+    (property "Sourcing" "JLCPCB" (id 7) (at 116.84 193.04 0)
+      (effects (font (size 1.27 1.27)) hide)
+    )
+    (property "SourcingPartNum" "C144397" (id 8) (at 116.84 193.04 0)
+      (effects (font (size 1.27 1.27)) hide)
+    )

Commit message: some minor attribute changes
Parts:
- U1: Manufacturer (none) -> STMicroelectronics; ManufacturerPartNum (none) -> ST1S14PHR; Sourcing (none) -> JLCPCB; SourcingPartNum (none) -> C84130; Umax (none) -> 48V
Changed lines of the file:
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@@
   (symbol (lib_id "Regulator_Switching:ST1S14PHR") (at 58.42 247.65 0) (unit 1)
     (in_bom yes) (on_board yes) (fields_autoplaced)
-    (property "Reference" "U1" (id 0) (at 58.42 234.95 0))
-    (property "Value" "ST1S14PHR" (id 1) (at 58.42 237.49 0))
+    (property "Reference" "U1" (id 0) (at 58.42 232.41 0))
+    (property "Value" "ST1S14PHR" (id 1) (at 58.42 234.95 0))
     (property "Footprint" "Package_SO:TI_SO-PowerPAD-8" (id 2) (at 61.595 256.54 0)
       (effects (font (size 1.27 1.27) italic) (justify left) hide)
@@
       (effects (font (size 1.27 1.27)) hide)
     )
+    (property "Manufacturer" "STMicroelectronics" (id 4) (at 58.42 247.65 0)
+      (effects (font (size 1.27 1.27)) hide)
+    )
+    (property "ManufacturerPartNum" "ST1S14PHR" (id 5) (at 58.42 247.65 0)
+      (effects (font (size 1.27 1.27)) hide)
+    )
+    (property "Sourcing" "JLCPCB" (id 6) (at 58.42 247.65 0)
+      (effects (font (size 1.27 1.27)) hide)
+    )
+    (property "SourcingPartNum" "C84130" (id 7) (at 58.42 247.65 0)
+      (effects (font (size 1.27 1.27)) hide)
+    )
+    (property "Umax" "48V" (id 8) (at 58.42 237.49 0))
     (pin "1")
     (pin "2")
